File: schematic/schematic.kicad_sch (KiCad schematic)
At the start: 15 parts, among them U1 STM32H743VITx

Commit message: vẽ xong phần cơ bản
Parts:
- added C14: 100nF, Capacitor_SMD:C_0805_2012Metric, symbol Device:C
- added C15: 0.1uF, Capacitor_SMD:C_0805_2012Metric, symbol Device:C
- added C16, C17: C, Capacitor_SMD:C_0805_2012Metric, symbol Device:C
- added J1: Conn_ARM_SWD_TagConnect_TC2030-NL, Connector:Tag-Connect_TC2030-IDC-NL_2x03_P1.27mm_Vertical, symbol Connector:Conn_ARM_SWD_TagConnect_TC2030-NL
- added R2, R3: 10K, Resistor_SMD:R_0805_2012Metric, symbol Device:R
- added SW1: SW_Push, Button_Switch_SMD:SW_Push_1P1T_NO_6x6mm_H9.5mm, symbol Switch:SW_Push
- added Y1: Crystal_GND23_Small, Crystal:Crystal_SMD_EuroQuartz_MJ-4Pin_5.0x3.2mm_HandSoldering, symbol Device:Crystal_GND23_Small
- R1: footprint (none) -> Resistor_SMD:R_0805_2012Metric
Connections:
- net +3V3: now also C15.1, J1.1 (VCC), R2.1
- net GND: now also C14.1, C15.2, C16.2, C17.2, J1.5 (GND), R3.2, SW1.1, Y1.2, Y1.3
- net NRST: now also C14.2, SW1.2
- net PH0: now reaches U1.12 (PH0)
- net PH0: now also C17.1, Y1.4
- net PH1: now reaches U1.13 (PH1)
- net PH1: now also C16.1, Y1.1
- net SWDIO: now reaches U1.72 (PA13)
- net SWDIO: now also J1.2 (SWDIO), R3.1
- net SWCLK: now reaches U1.76 (PA14)
- net SWCLK: now also J1.4 (SWCLK), R2.2
Other:
- note added: "Button reset"
- note added: "Crystal"
- note added: "Debug"
- moved on the sheet: C10, C11

Commit message: no message
Parts:
- added C18: 680uF, symbol Device:C
- added C19: 220uF, symbol Device:C
- added C20: 0.33uF, symbol Device:C
- added C22: 100nF, symbol Device:C
- added C23, C24: 10uF, symbol Device:C
- added R4, R5: 200K, symbol Device:R
- added R6: 1ohm, symbol Device:R
- added U2: AMS1117, Package_TO_SOT_SMD:SOT-223-3_TabPin2, symbol Regulator_Linear:AMS1117
- added U3: LM2596S-5, Package_TO_SOT_SMD:TO-263-5_TabPin3, symbol Regulator_Switching:LM2596S-5
- added U5: L7805, symbol Regulator_Linear:L7806
Connections:
- net +3V3: now also C24.1, U2.2 (VO)
- net GND: now also C18.2, C19.2, C20.2, C22.2, C23.2, C24.2, R4.2, U2.1 (ADJ), U3.3 (GND), U3.5 (~{ON}/OFF), U5.2 (GND)
- new net: C18.1, R4.1, R5.2, U3.1 (VIN)
- new net: C20.1, R6.1, U5.1 (IN)
- new net +24V: R5.1
- new net +5V: C19.1, C22.1, C23.1, U2.3 (VI), U3.2 (OUT), U3.4 (FB), U5.3 (OUT)
- new net +7.5V: R6.2
Other:
- note added: "+3V3"
- note added: "+5V"

Commit message: no message
Parts:
- removed C19: 220uF, symbol Device:C
- removed C20: 0.33uF, symbol Device:C
- removed C22: 100nF, symbol Device:C
- removed R6: 1ohm, symbol Device:R
- removed U3: LM2596S-5, Package_TO_SOT_SMD:TO-263-5_TabPin3, symbol Regulator_Switching:LM2596S-5
- removed U5: L7805, symbol Regulator_Linear:L7806
- added D1: D, symbol Device:D
- added L1: L, symbol Device:L
- added U4: MP1584, MP1584:SO-08POWER, symbol mp1584:MP1584
- C18: value 680uF -> C
- R4, R5: value 200K -> R
Connections:
- net +24V is gone; now on net GND: R5.1
- net +5V: now also C18.1, R4.1, L1.2
- net GND: now also D1.2 (A); no longer R4.2
- new net: D1.1 (K), L1.1, U4.1 (SW)
- new net: R4.2, R5.2, U4.4 (FB)
Other:
- note removed: "+5V"

Commit message: no message
Parts:
- added C19: 10uF, symbol Device:C
- added C20: 100nF, symbol Device:C
- C18: value C -> 22uF
- D1: value D -> 40V-3A
- L1: value L -> 10uH
- R4: value R -> 210K
- R5: value R -> 40.2K
Connections:
- net GND: now also C19.1
- net at D1.1 (K), L1.1, U4.1 (SW): now also C20.2
- net +7.5V: now reaches U4.7 (VIN)
- net +7.5V: now also C19.2
- net at U4.8 (BST): now also C20.1

Commit message: thêm phần driver tb66, ve phần nguồn 5v
Parts:
- added C21: 150pF, Capacitor_SMD:C_0805_2012Metric, symbol Device:C
- added C22, C27: 100nF, symbol Device:C
- added C25, C26: 10uF, symbol Device:C_Polarized
- added R6: 100k, Resistor_SMD:R_0805_2012Metric, symbol Device:R
- added R7: 100K, Resistor_SMD:R_0805_2012Metric, symbol Device:R
- added R8: 67k, Resistor_SMD:R_0805_2012Metric, symbol Device:R
- added R9: 20k, Resistor_SMD:R_0805_2012Metric, symbol Device:R
- added U3: TB6612FNG_C_8_EL, Library:SOP65P760X160-24N, symbol TB6612FNG_C_8_EL:TB6612FNG_C_8_EL
- C18, C19, C20, C23, C24: footprint (none) -> Capacitor_SMD:C_0805_2012Metric
- D1: footprint (none) -> Diode_SMD:D_2010_5025Metric_Pad1.52x2.65mm_HandSolder
- L1: value 10uH -> 15uH; footprint (none) -> Inductor_SMD:L_12x12mm_H4.5mm
- R4, R5: footprint (none) -> Resistor_SMD:R_0805_2012Metric
Connections:
- net +5V: now also C26.1, C27.1, U3.13 (VM2), U3.14 (VM3), U3.24 (VM1)
- net GND: now also U4.5 (GND), C22.2, C25.2, C26.2, C27.2, R6.2, R7.2, R9.2, U3.10 (PGND2@2), U3.18 (GND), U3.3 (PGND1@1), U3.4 (PGND1@2), U3.9 (PGND2@1)
- net BIN1: now reaches U1.87 (PD6)
- net BIN1: now also U3.17 (BIN1)
- net BIN2: now reaches U1.88 (PD7)
- net BIN2: now also U3.16 (BIN2)
- net AIN1: now reaches U1.91 (PB5)
- net AIN1: now also U3.21 (AIN1)
- net AIN2: now reaches U1.92 (PB6)
- net AIN2: now also U3.22 (AIN2)
- net at U4.2 (EN): now also R8.2, R9.1
- net at U4.3 (COMP): now also C21.1
- net at U4.6 (FREQ): now also R6.1
- net +7.5V renamed 6-7.5V
- net 6-7.5V: now also R8.1
- new net: C21.2, R7.1
- new net +3.3V: C22.1, C25.1, U3.19 (STBY), U3.20 (VCC)
Other:
- note added: "5V"
- moved on the sheet: C18, C19, C20, D1, L1, R4, R5, U4

Commit message: no message
Parts:
- C1, C10, C11, C12, C13, C14, C15, C18, C19, C2, C20, C24, C3, C4, C5, C6, C7, C8, C9: footprint Capacitor_SMD:C_0805_2012Metric -> Capacitor_SMD:C_0603_1608Metric
- C16, C17: value C -> 15pF; footprint Capacitor_SMD:C_0805_2012Metric -> Capacitor_SMD:C_0603_1608Metric
- C22, C25, C26, C27: footprint (none) -> Capacitor_SMD:C_0603_1608Metric
- D1: value 40V-3A -> 40V-5A; footprint Diode_SMD:D_2010_5025Metric_Pad1.52x2.65mm_HandSolder -> Diode_SMD:D_SMA
- L1: footprint Inductor_SMD:L_12x12mm_H4.5mm -> Inductor_SMD:L_7.3x7.3_H4.5
- R1, R2, R3, R4, R6, R7: footprint Resistor_SMD:R_0805_2012Metric -> Resistor_SMD:R_0603_1608Metric
- R8: value 67k -> 63.4K
- SW1: footprint Button_Switch_SMD:SW_Push_1P1T_NO_6x6mm_H9.5mm -> Button_Switch_SMD:SW_Push_1P1T_NO_CK_KSC6xxJ
Connections:
- net Encoder_A_R: now reaches U1.22 (PA0)
- net Encoder_B_R: now reaches U1.23 (PA1)
- net Encoder_A_L: now reaches U1.29 (PA5)
- net sensorFF: now reaches U1.30 (PA6)
- net sensorFR: now reaches U1.31 (PA7)
- net sensorFL: now reaches U1.32 (PC4)
- net sensorR: now reaches U1.33 (PC5)
- net sensorL: now reaches U1.35 (PB1)
- net PWMA: now reaches U1.39 (PE9)
- net PWMA: now also U3.23 (PWMA)
- net PWMB: now reaches U1.41 (PE11)
- net PWMB: now also U3.15 (PWMB)
- net UART3_TX: now reaches U1.46 (PB10)
- net UART3_RX: now reaches U1.47 (PB11)
- net UART1_TX: now reaches U1.53 (PB14)
- net UART1_RX: now reaches U1.54 (PB15)
- net Encoder_B_L: now reaches U1.89 (PB3)
- net at U3.1 (AO1@1): now also U3.2 (AO1@2)
- net at U3.11 (BO1@1): now also U3.12 (BO1@2)
- net at U3.5 (AO2@1): now also U3.6 (AO2@2)
- net at U3.7 (BO2@1): now also U3.8 (BO2@2)

Commit message: xong phần nguồn
Parts:
- R8: value 63.4K -> 75k
Connections:
- net 6-7.5V renamed 6.5-7.5V
Changed lines of the file:
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@@
 	(text "5V"
 		(exclude_from_sim no)
-		(at 1079.754 134.62 0)
+		(at 1075.69 136.144 0)
 		(effects
 			(font
@@
 			)
 		)
-		(property "Value" "63.4K"
+		(property "Value" "75k"
 			(at 1096.772 92.71 0)
 			(effects
@@
 		(on_board yes)
 		(dnp no)
-		(fields_autoplaced yes)
 		(property "Reference" "#PWR022"
 			(at 1101.09 87.63 0)
@@
 			)
 		)
-		(property "Value" "6-7.5V"
-			(at 1093.47 87.6299 90)
+		(property "Value" "6.5-7.5V"
+			(at 1088.136 87.63 90)
 			(effects
 				(font
 					(size 1.27 1.27)
 				)
-				(justify left)
 			)
 		)
