File: schematic/schematic.kicad_sch (KiCad schematic)
At the start: 45 parts, among them J2 Conn_01x04_Socket, SW1 SW_Push, U1 STM32H743VITx, U2 AMS1117, U3 TB6612FNG_C_8_EL, U4 MP1584, Y1 Crystal_GND23_Small

Commit message: vẽ đủ đò ăn chơi chưa duyệt
Parts:
- added BZ1: Buzzer, Buzzer_Beeper:MagneticBuzzer_CUI_CMT-8504-100-SMT, symbol Device:Buzzer
- added D2, D3, D4, D5, D6, D7: LED, LED_SMD:LED_0603_1608Metric, symbol Device:LED
- added J1, J3, J4: Conn_01x04_Socket, Connector_JST:JST_PH_B4B-PH-K_1x04_P2.00mm_Vertical, symbol Connector:Conn_01x04_Socket
- added J10, J11: Conn_01x06_Pin, Connector_JST:JST_PH_S6B-PH-K_1x06_P2.00mm_Horizontal, symbol Connector:Conn_01x06_Pin
- added J5, J6, J7: Conn_01x03_Pin, Connector_JST:JST_PH_S3B-PH-K_1x03_P2.00mm_Horizontal, symbol Connector:Conn_01x03_Pin
- added J8, J9: Conn_01x03_Pin, Connector_JST:JST_PH_B3B-PH-K_1x03_P2.00mm_Vertical, symbol Connector:Conn_01x03_Pin
- added Q1: S8550, Package_TO_SOT_SMD:SOT-23, symbol Transistor_BJT:S8550
- added R10, R11, R12, R13, R14, R15, R16: 1K, Resistor_SMD:R_0603_1608Metric, symbol Device:R
- Y1: footprint Crystal:Crystal_SMD_EuroQuartz_MJ-4Pin_5.0x3.2mm_HandSoldering -> Crystal:Crystal_SMD_3225-4Pin_3.2x2.5mm
Connections:
- net +3.3V is gone; now on net +3V3: C22.1, C25.1, U3.19 (STBY), U3.20 (VCC)
- net +3V3: now also J1.1 (Pin_1), J3.1 (Pin_1), Q1.1 (E), R11.1
- net +5V: now also J10.1 (Pin_1), J11.1 (Pin_1), J5.3 (Pin_3), J6.3 (Pin_3), J7.3 (Pin_3), J8.3 (Pin_3), J9.3 (Pin_3)
- net Encoder_A_L: now also J11.4 (Pin_4)
- net Encoder_A_R: now also J10.3 (Pin_3)
- net Encoder_B_L: now also J11.3 (Pin_3)
- net Encoder_B_R: now also J10.4 (Pin_4)
- net GND: now also BZ1.2 (-), D2.1 (K), D3.1 (K), D4.1 (K), D5.1 (K), D6.1 (K), D7.1 (K), J1.4 (Pin_4), J10.2 (Pin_2), J11.2 (Pin_2), J3.4 (Pin_4), J4.4 (Pin_4), J5.1 (Pin_1), J6.1 (Pin_1), J7.1 (Pin_1), J8.1 (Pin_1), J9.1 (Pin_1)
- net UART1_RX: now also J3.2 (Pin_2)
- net UART1_TX: now also J3.3 (Pin_3)
- net UART3_RX: now also U1.56 (PD9), J1.2 (Pin_2); no longer U1.47 (PB11)
- net UART3_TX: now also U1.55 (PD8), J1.3 (Pin_3); no longer U1.46 (PB10)
- net sensorFF: now also J5.2 (Pin_2)
- net sensorFL: now also J7.2 (Pin_2)
- net sensorFR: now also J6.2 (Pin_2)
- net sensorL: now also J8.2 (Pin_2)
- net sensorR: now also J9.2 (Pin_2)
- net LED_L: now reaches U1.63 (PC6)
- net LED_L: now also R16.1
- net LED_R: now reaches U1.64 (PC7)
- net LED_R: now also R15.1
- net LED_FL: now reaches U1.65 (PC8)
- net LED_FL: now also R14.1
- net LED_FR: now reaches U1.66 (PC9)
- net LED_FR: now also R12.1
- net LED_FF: now reaches U1.67 (PA8)
- net LED_FF: now also R13.1
- net BUZZ: now reaches U1.68 (PA9)
- net BUZZ: now also R10.2
- net M1-R: now reaches U3.1 (AO1@1), U3.2 (AO1@2)
- net M1-R: now also J10.6 (Pin_6)
- net M2-R: now reaches U3.11 (BO1@1), U3.12 (BO1@2)
- net M2-R: now also J11.6 (Pin_6)
- net M1-L: now reaches U3.5 (AO2@1), U3.6 (AO2@2)
- net M1-L: now also J10.5 (Pin_5)
- net M2-L: now reaches U3.7 (BO2@1), U3.8 (BO2@2)
- net M2-L: now also J11.5 (Pin_5)
- new net: D3.2 (A), R12.2
- new net: Q1.2 (B), R10.1
- new net: BZ1.1 (+), Q1.3 (C)
- new net: D2.2 (A), R11.2
- new net: D6.2 (A), R15.2
- new net: D5.2 (A), R14.2
- new net: D7.2 (A), R16.2
- new net: D4.2 (A), R13.2
- new net 5V: J4.1 (Pin_1)
- new net I2C2_SCL: J4.3 (Pin_3), U1.46 (PB10)
- new net I2C2_SDA: J4.2 (Pin_2), U1.47 (PB11)
Other:
- note added: "BUZZER"
- note added: "Driver"
- note added: "I2C"
- note added: "LED_Debug"
- note added: "MPU Sensor"
- note added: "Sensor-header"
- note added: "UART1"
- note added: "header-motor-encoder"
- moved on the sheet: C18, C19, C20, C21, D1, L1, R4, R5, R6, R7, R8, R9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

Commit message: thếu nút nhấn
Parts:
- added R17, R18: 4.7k, Resistor_SMD:R_0603_1608Metric, symbol Device:R
Connections:
- net +3V3: now also R17.1, R18.1
- net I2C2_SCL: now also R18.2
- net I2C2_SDA: now also R17.2
- net Encoder_A_L renamed EN_A_L
- net Encoder_A_R renamed EN_A_R
- net Encoder_B_L renamed EN_B_L
- net Encoder_B_R renamed EN_B_R
- net sensorFF renamed SS_FF
- net sensorFL renamed SS_FL
- net sensorFR renamed SS_FR
- net sensorL renamed SS_L
- net sensorR renamed SS_R
Other:
- moved on the sheet: J4

Commit message: no message
Parts:
- added C28, C29: 100nF, Capacitor_SMD:C_0603_1608Metric, symbol Device:C
- added R19, R20: 1k, Resistor_SMD:R_0603_1608Metric, symbol Device:R
- added SW2, SW3: SW_Push, Button_Switch_SMD:SW_Tactile_SPST_NO_Straight_CK_PTS636Sx25SMTRLFS, symbol Switch:SW_Push
- SW1: footprint Button_Switch_SMD:SW_Push_1P1T_NO_CK_KSC6xxJ -> Button_Switch_SMD:SW_Tactile_SPST_NO_Straight_CK_PTS636Sx25SMTRLFS
Connections:
- net +3V3: now also C28.1, C29.1, R19.1, R20.1
- net GND: now also C28.2, C29.2, SW2.1, SW3.1
- net BUTTON_0: now reaches U1.82 (PD1)
- net BUTTON_0: now also R19.2, SW3.2
- net BUTTON_1: now reaches U1.83 (PD2)
- net BUTTON_1: now also R20.2, SW2.2
Other:
- note added: "User button"

Commit message: trc khi xoá ve lai
Parts:
- added J12: Conn_01x02_Socket, Connector_JST:JST_XA_B02B-XASK-1_1x02_P2.50mm_Vertical, symbol Connector:Conn_01x02_Socket
Connections:
- net 5V is gone; now on net +5V: J4.1 (Pin_1)
- net 6.5-7.5V: now also J12.1 (Pin_1)
- net EN_A_L: now also J10.4 (Pin_4); no longer J11.4 (Pin_4)
- net EN_A_R: now also J11.3 (Pin_3); no longer J10.3 (Pin_3)
- net EN_B_L: now also J10.3 (Pin_3); no longer J11.3 (Pin_3)
- net EN_B_R: now also J11.4 (Pin_4); no longer J10.4 (Pin_4)
- net GND: now also J12.2 (Pin_2)
- net M1-L: now also J10.6 (Pin_6); no longer J10.5 (Pin_5)
- net M1-R: now also J10.5 (Pin_5); no longer J10.6 (Pin_6)
Changed lines of the file:
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@@
 	(wire
 		(pts
+			(xy 1068.07 233.68) (xy 1070.61 233.68)
+		)
+		(stroke
+			(width 0)
+			(type default)
+		)
+	)
+	(wire
+		(pts
 			(xy 660.4 464.82) (xy 666.75 464.82)
 		)
@@
 	(wire
 		(pts
+			(xy 1068.07 236.22) (xy 1070.61 236.22)
+		)
+		(stroke
+			(width 0)
+			(type default)
+		)
+	)
+	(wire
+		(pts
 			(xy 1002.03 96.52) (xy 1007.11 96.52)
 		)
@@
 	)
 	(rectangle
+		(start 1038.225 216.535)
+		(end 1103.63 258.445)
+		(stroke
+			(width 0)
+			(type default)
+		)
+		(fill
+			(type none)
+		)
+	)
+	(rectangle
 		(start 1042.67 11.43)
 		(end 1111.25 59.69)
@@
 	)
 	(label "EN_B_R"
-		(at 1155.7 195.58 180)
+		(at 1120.14 195.58 180)
 		(fields_autoplaced yes)
 		(effects
@@
 	)
 	(label "EN_B_L"
-		(at 1120.14 198.12 180)
+		(at 1155.7 198.12 180)
 		(fields_autoplaced yes)
 		(effects
@@
 	)
 	(label "EN_A_L"
-		(at 1120.14 195.58 180)
+		(at 1155.7 195.58 180)
 		(fields_autoplaced yes)
 		(effects
@@
 	)
 	(label "M1-R"
-		(at 1155.7 190.5 0)
+		(at 1155.7 193.04 0)
 		(fields_autoplaced yes)
 		(effects
@@
 	)
 	(label "M1-L"
-		(at 1155.7 193.04 0)
+		(at 1155.7 190.5 0)
 		(fields_autoplaced yes)
 		(effects
@@
 	)
 	(label "EN_A_R"
-		(at 1155.7 198.12 180)
+		(at 1120.14 198.12 180)
 		(fields_autoplaced yes)
 		(effects
@@
 	)
 	(symbol
-		(lib_id "power:+3.3V")
-		(at 1076.96 154.94 0)
-		(unit 1)
-		(exclude_from_sim no)
-		(in_bom yes)
-		(on_board yes)
-		(dnp no)
-		(fields_autoplaced yes)
-		(property "Reference" "#PWR039"
-			(at 1076.96 158.75 0)
-			(effects
-				(font
-					(size 1.27 1.27)
-				)
-				(hide yes)
-			)
-		)
-		(property "Value" "5V"
-			(at 1076.96 149.86 0)
-			(effects
-				(font
-					(size 1.27 1.27)
-				)
-			)
-		)
-		(property "Footprint" ""
-			(at 1076.96 154.94 0)
-			(effects
-				(font
-					(size 1.27 1.27)
-				)
-				(hide yes)
-			)
-		)
-		(property "Datasheet" ""
-			(at 1076.96 154.94 0)
-			(effects
-				(font
-					(size 1.27 1.27)
-				)
-				(hide yes)
-			)
-		)
-		(property "Description" "Power symbol creates a global label with name \"+3.3V\""
-			(at 1076.96 154.94 0)
-			(effects
-				(font
-					(size 1.27 1.27)
-				)
-				(hide yes)
-			)
-		)
-		(pin "1"
-		)
-		(instances
-			(project "schematic"
-				(path "/294fb569-9d7c-450c-aa5f-45fbbde8417a"
-					(reference "#PWR039")
-					(unit 1)
-				)
-			)
-		)
-	)
-	(symbol
 		(lib_id "power:+5V")
 		(at 1052.83 80.01 270)
@@
 	)
 	(symbol
+		(lib_id "power:+7.5V")
+		(at 1068.07 233.68 90)
+		(unit 1)
+		(exclude_from_sim no)
+		(in_bom yes)
+		(on_board yes)
+		(dnp no)
+		(property "Reference" "#PWR064"
+			(at 1071.88 233.68 0)
+			(effects
+				(font
+					(size 1.27 1.27)
+				)
+				(hide yes)
+			)
+		)
+		(property "Value" "6.5-7.5V"
+			(at 1058.926 233.68 90)
+			(effects
+				(font
+					(size 1.27 1.27)
+				)
+			)
+		)
+		(property "Footprint" ""
+			(at 1068.07 233.68 0)
+			(effects
+				(font
+					(size 1.27 1.27)
+				)
+				(hide yes)
+			)
+		)
+		(property "Datasheet" ""
+			(at 1068.07 233.68 0)
+			(effects
+				(font
+					(size 1.27 1.27)
+				)
+				(hide yes)
+			)
+		)
+		(property "Description" "Power symbol creates a global label with name \"+7.5V\""
+			(at 1068.07 233.68 0)
+			(effects
+				(font
+					(size 1.27 1.27)
+				)
+				(hide yes)
+			)
+		)
+		(pin "1"
+		)
+		(instances
+			(project "schematic"
+				(path "/294fb569-9d7c-450c-aa5f-45fbbde8417a"
+					(reference "#PWR064")
+					(unit 1)
+				)
+			)
+		)
+	)
+	(symbol
 		(lib_id "power:GND")
 		(at 571.5 356.87 270)
@@
 	)
 	(symbol
+		(lib_id "Connector:Conn_01x02_Socket")
+		(at 1075.69 233.68 0)
+		(unit 1)
+		(exclude_from_sim no)
+		(in_bom yes)
+		(on_board yes)
+		(dnp no)
+		(fields_autoplaced yes)
+		(property "Reference" "J12"
+			(at 1076.96 233.6799 0)
+			(effects
+				(font
+					(size 1.27 1.27)
+				)
+				(justify left)
+			)
+		)
+		(property "Value" "Conn_01x02_Socket"
+			(at 1076.96 236.2199 0)
+			(effects
+				(font
+					(size 1.27 1.27)
+				)
+				(justify left)
+			)
+		)
+		(property "Footprint" "Connector_JST:JST_XA_B02B-XASK-1_1x02_P2.50mm_Vertical"
+			(at 1075.69 233.68 0)
+			(effects
+				(font
+					(size 1.27 1.27)
+				)
+				(hide yes)
+			)
+		)
+		(property "Datasheet" "~"
+			(at 1075.69 233.68 0)
+			(effects
+				(font
+					(size 1.27 1.27)
+				)
+				(hide yes)
+			)
+		)
+		(property "Description" "Generic connector, single row, 01x02, script generated"
+			(at 1075.69 233.68 0)
+			(effects
+				(font
+					(size 1.27 1.27)
+				)
+				(hide yes)
+			)
+		)
+		(pin "1"
+		)
+		(pin "2"
+		)
+		(instances
+			(project ""
+				(path "/294fb569-9d7c-450c-aa5f-45fbbde8417a"
+					(reference "J12")
+					(unit 1)
+				)
+			)
+		)
+	)
+	(symbol
 		(lib_id "power:+5V")
 		(at 1024.89 158.75 0)
@@
 	(symbol
 		(lib_id "power:+5V")
+		(at 1076.96 154.94 0)
+		(unit 1)
+		(exclude_from_sim no)
+		(in_bom yes)
+		(on_board yes)
+		(dnp no)
+		(fields_autoplaced yes)
+		(property "Reference" "#PWR039"
+			(at 1076.96 158.75 0)
+			(effects
+				(font
+					(size 1.27 1.27)
+				)
+				(hide yes)
+			)
+		)
+		(property "Value" "+5V"
+			(at 1076.96 149.86 0)
+			(effects
+				(font
+					(size 1.27 1.27)
+				)
+			)
+		)
+		(property "Footprint" ""
+			(at 1076.96 154.94 0)
+			(effects
+				(font
+					(size 1.27 1.27)
+				)
+				(hide yes)
+			)
+		)
+		(property "Datasheet" ""
+			(at 1076.96 154.94 0)
+			(effects
+				(font
+					(size 1.27 1.27)
+				)
+				(hide yes)
+			)
+		)
+		(property "Description" "Power symbol creates a global label with name \"+5V\""
+			(at 1076.96 154.94 0)
+			(effects
+				(font
+					(size 1.27 1.27)
+				)
+				(hide yes)
+			)
+		)
+		(pin "1"
+		)
+		(instances
+			(project "schematic"
+				(path "/294fb569-9d7c-450c-aa5f-45fbbde8417a"
+					(reference "#PWR039")
+					(unit 1)
+				)
+			)
+		)
+	)
+	(symbol
+		(lib_id "power:+5V")
 		(at 1159.51 86.36 270)
 		(unit 1)
@@
 					(unit 1)
 				)
+			)
+		)
+	)
+	(symbol
+		(lib_id "power:GND")
+		(at 1068.07 236.22 0)
+		(unit 1)
+		(exclude_from_sim no)
+		(in_bom yes)
+		(on_board yes)
+		(dnp no)
+		(fields_autoplaced yes)
+		(property "Reference" "#PWR065"
+			(at 1068.07 242.57 0)
+			(effects
+				(font
+					(size 1.27 1.27)
+				)
+				(hide yes)
+			)
+		)
+		(property "Value" "GND"
+			(at 1068.07 241.3 0)
+			(effects
+				(font
+					(size 1.27 1.27)
+				)
+			)
+		)
+		(property "Footprint" ""
+			(at 1068.07 236.22 0)
+			(effects
+				(font
+					(size 1.27 1.27)
+				)
+				(hide yes)
+			)
+		)
+		(property "Datasheet" ""
+			(at 1068.07 236.22 0)
+			(effects
+				(font
+					(size 1.27 1.27)
+				)
+				(hide yes)
+			)
+		)
+		(property "Description" "Power symbol creates a global label with name \"GND\" , ground"
+			(at 1068.07 236.22 0)
+			(effects
+				(font
+					(size 1.27 1.27)
+				)
+				(hide yes)
+			)
+		)
+		(pin "1"
+		)
+		(instances
+			(project ""
+				(path "/294fb569-9d7c-450c-aa5f-45fbbde8417a"
+					(reference "#PWR065")
+					(unit 1)
+				)

Commit message: 1
Parts:
- removed J3: Conn_01x04_Socket, Connector_JST:JST_PH_B4B-PH-K_1x04_P2.00mm_Vertical, symbol Connector:Conn_01x04_Socket
- removed R12, R13, R14, R15, R16: 1K, Resistor_SMD:R_0603_1608Metric, symbol Device:R
- added C30, C31: 22uF, Capacitor_SMD:C_0201_0603Metric, symbol Device:C
- added R21: 1.1R, Resistor_SMD:R_0805_2012Metric, symbol Device:R
- added RN1: R_Network05, Resistor_SMD:R_Array_Convex_5x0603, symbol Device:R_Network05
- added RN2: R_Pack05, Resistor_SMD:R_Array_Convex_5x0603, symbol Device:R_Pack05
- added SW4: SW_DIP_x05, Button_Switch_SMD:SW_DIP_SPSTx05_Slide_KingTek_DSHP05TS_W7.62mm_P1.27mm, symbol Switch:SW_DIP_x05
- added U5: AMS1117-5.0, Package_TO_SOT_SMD:SOT-223-3_TabPin2, symbol Regulator_Linear:AMS1117-5.0
- J1, J4: footprint Connector_JST:JST_PH_B4B-PH-K_1x04_P2.00mm_Vertical -> Connector_PinHeader_2.54mm:PinHeader_1x04_P2.54mm_Vertical
- J10, J11: footprint Connector_JST:JST_PH_S6B-PH-K_1x06_P2.00mm_Horizontal -> JST-254:JST 6
- J2: footprint Connector_JST:JST_PH_B4B-PH-K_1x04_P2.00mm_Vertical -> Connector_JST:JST_SH_BM04B-SRSS-TB_1x04-1MP_P1.00mm_Vertical
- J5, J6, J7: footprint Connector_JST:JST_PH_S3B-PH-K_1x03_P2.00mm_Horizontal -> Connector_PinHeader_2.54mm:PinHeader_1x03_P2.54mm_Vertical
- J8, J9: footprint Connector_JST:JST_PH_B3B-PH-K_1x03_P2.00mm_Vertical -> Connector_PinHeader_2.54mm:PinHeader_1x03_P2.54mm_Vertical
Connections:
- net +3V3: now also RN2.1 (R1.1), RN2.2 (R2.1), RN2.3 (R3.1), RN2.4 (R4.1), RN2.5 (R5.1)
- net +5V: now also C30.1, U5.2 (VO)
- net BIN1: now also U1.88 (PD7); no longer U1.87 (PD6)
- net BIN2: now also U1.87 (PD6); no longer U1.88 (PD7)
- net BUTTON_0: now also U1.24 (PA2); no longer U1.82 (PD1)
- net BUTTON_1: now also U1.25 (PA3); no longer U1.83 (PD2)
- net BUZZ: now also U1.61 (PD14); no longer U1.68 (PA9)
- net EN_A_L: now also U1.77 (PA15); no longer U1.29 (PA5)
- net GND: now also C30.2, C31.2, RN1.1 (common), U5.1 (GND); no longer D3.1 (K), D4.1 (K), D5.1 (K), D6.1 (K), D7.1 (K)
- net LED_FF: now also D5.2 (A), U1.64 (PC7); no longer U1.67 (PA8)
- net LED_FL: now also D3.2 (A), U1.63 (PC6); no longer U1.65 (PC8)
- net LED_FR: now also D6.2 (A), U1.65 (PC8); no longer U1.66 (PC9)
- net LED_L: now also D4.2 (A), U1.62 (PD15); no longer U1.63 (PC6)
- net LED_R: now also D7.2 (A), U1.66 (PC9); no longer U1.64 (PC7)
- net M1-L: now also J11.6 (Pin_6); no longer J10.6 (Pin_6)
- net M1-R: now also J11.5 (Pin_5); no longer J10.5 (Pin_5)
- net M2-L: now also J10.5 (Pin_5); no longer J11.5 (Pin_5)
- net M2-R: now also J10.6 (Pin_6); no longer J11.6 (Pin_6)
- net PWMA: now also U1.67 (PA8); no longer U1.39 (PE9)
- net PWMB: now also U1.68 (PA9); no longer U1.41 (PE11)
- net BIT_SW_4: now reaches U1.1 (PE2)
- net BIT_SW_4: now also SW4.6
- net BIT_SW_3: now reaches U1.2 (PE3)
- net BIT_SW_3: now also SW4.7
- net BIT_SW_2: now reaches U1.3 (PE4)
- net BIT_SW_2: now also SW4.8
- net BIT_SW_1: now reaches U1.4 (PE5)
- net BIT_SW_1: now also SW4.9
- net BIT_SW_0: now reaches U1.5 (PE6)
- net BIT_SW_0: now also SW4.10
- net UART1_RX: no longer names the net of U1.54 (PB15)
- net UART1_TX: no longer names the net of U1.53 (PB14)
- new net: D4.1 (K), RN1.2 (R1)
- new net: D3.1 (K), RN1.3 (R2)
- new net: D5.1 (K), RN1.4 (R3)
- new net: D6.1 (K), RN1.5 (R4)
- new net: D7.1 (K), RN1.6 (R5)
- new net: RN2.10 (R1.2), SW4.1
- new net: RN2.6 (R5.2), SW4.5
- new net: RN2.7 (R4.2), SW4.4
- new net: RN2.8 (R3.2), SW4.3
- new net: RN2.9 (R2.2), SW4.2
- new net: C31.1, R21.2, U5.3 (VI)
- new net +7.5V: R21.1
Other:
- note removed: "UART1"
- moved on the sheet: D3, D4, D5, D6, D7, J1

Commit message: gần hoàn thiện pcb
Parts:
- removed D6, D7: LED, LED_SMD:LED_0603_1608Metric, symbol Device:LED
- removed J5, J6, J7, J8, J9: Conn_01x03_Pin, Connector_PinHeader_2.54mm:PinHeader_1x03_P2.54mm_Vertical, symbol Connector:Conn_01x03_Pin
- added C32: 10uF, Capacitor_Tantalum_SMD:CP_EIA-3216-10_Kemet-I, symbol Device:C_Polarized
- added D8, D9: LED, LED_SMD:LED_0603_1608Metric, symbol Device:LED
- added J5: Conn_01x07_Pin, Connector_PinHeader_2.54mm:PinHeader_1x07_P2.54mm_Vertical, symbol Connector:Conn_01x07_Pin
- C25, C26: footprint Capacitor_SMD:C_0603_1608Metric -> Capacitor_Tantalum_SMD:CP_EIA-3216-10_Kemet-I
- J1, J4: footprint Connector_PinHeader_2.54mm:PinHeader_1x04_P2.54mm_Vertical -> JST-254:JST 4
- J10, J11: footprint JST-254:JST 6 -> Connector_JST:JST_SH_BM06B-SRSS-TB_1x06-1MP_P1.00mm_Vertical
- J2: footprint Connector_JST:JST_SH_BM04B-SRSS-TB_1x04-1MP_P1.00mm_Vertical -> JST-254:JST 4
Connections:
- net +7.5V is gone; now on net 6.5-7.5V: R21.1
- net +5V: now also C32.1, J5.7 (Pin_7)
- net BIT_SW_0: now also U1.1 (PE2); no longer U1.5 (PE6)
- net BIT_SW_1: now also U1.2 (PE3); no longer U1.4 (PE5)
- net BIT_SW_3: now also U1.4 (PE5); no longer U1.2 (PE3)
- net BIT_SW_4: now also U1.5 (PE6); no longer U1.1 (PE2)
- net GND: now also C32.2, J5.6 (Pin_6)
- net LED_FL: now also U1.62 (PD15); no longer U1.63 (PC6)
- net LED_FR: now also D9.2 (A)
- net LED_L: now also U1.63 (PC6); no longer U1.62 (PD15)
- net LED_R: now also D8.2 (A)
- net M1-L: now also J11.5 (Pin_5); no longer J11.6 (Pin_6)
- net M1-R: now also J11.6 (Pin_6); no longer J11.5 (Pin_5)
- net M2-L: now also J10.6 (Pin_6); no longer J10.5 (Pin_5)
- net M2-R: now also J10.5 (Pin_5); no longer J10.6 (Pin_6)
- net SS_FF: now also J5.5 (Pin_5)
- net SS_FL: now also J5.3 (Pin_3)
- net SS_FR: now also J5.4 (Pin_4)
- net SS_L: now also J5.1 (Pin_1)
- net SS_R: now also J5.2 (Pin_2)
- net at RN1.5 (R4): now also D8.1 (K)
- net at RN1.6 (R5): now also D9.1 (K)
Other:
- moved on the sheet: BZ1, C1, C10, C11, C12, C13, C14, C15, C16, C17, C18, C19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

Commit message: cho doi xi va
Parts:
- removed C23: 10uF, Capacitor_SMD:C_0805_2012Metric, symbol Device:C
- removed C24: 10uF, Capacitor_SMD:C_0603_1608Metric, symbol Device:C
- removed C30, C31: 22uF, Capacitor_SMD:C_0201_0603Metric, symbol Device:C
- added C23, C24, C30, C31: 22uF, Capacitor_Tantalum_SMD:CP_EIA-3216-10_Kemet-I, symbol Device:C_Polarized
Connections:
- net +3V3: now also C24.1
- net +5V: now also C23.1, C30.1
- net GND: now also C23.2, C24.2, C30.2, C31.2
- net at R21.2, U5.3 (VI): now also C31.1

Commit message: khá ổn chờ chốt
Parts:
- removed BZ1: Buzzer, Buzzer_Beeper:MagneticBuzzer_CUI_CMT-8504-100-SMT, symbol Device:Buzzer
- removed RN1: R_Network05, Resistor_SMD:R_Array_Convex_5x0603, symbol Device:R_Network05
- added LS1: CMT-8530S-SMT, Buzzer_Beeper:CUI_CMT-8530S-SMT, symbol CMT-8530S-SMT:CMT-8530S-SMT
- added RN3: R_Pack05, Resistor_SMD:R_Array_Convex_5x0603, symbol Device:R_Pack05
- J12: footprint Connector_JST:JST_XA_B02B-XASK-1_1x02_P2.50mm_Vertical -> Connector_PinHeader_2.54mm:jst
- renumbered D9 to D3, D3 to D9
Connections:
- net +3V3: now also J10.1 (Pin_1), J11.1 (Pin_1), J4.1 (Pin_1)
- net +5V: no longer J10.1 (Pin_1), J11.1 (Pin_1), J4.1 (Pin_1)
- net EN_A_R: now also J11.4 (Pin_4); no longer J11.3 (Pin_3)
- net EN_B_R: now also J11.3 (Pin_3); no longer J11.4 (Pin_4)
- net GND: now also LS1.N, RN3.10 (R1.2), RN3.6 (R5.2), RN3.7 (R4.2), RN3.8 (R3.2), RN3.9 (R2.2)
- net LED_FL: now also D3.2 (A), U1.65 (PC8); no longer D9.2 (A), U1.62 (PD15)
- net LED_FR: now also D4.2 (A), U1.63 (PC6); no longer D3.2 (A), U1.65 (PC8)
- net LED_L: now also D8.2 (A), U1.66 (PC9); no longer D4.2 (A), U1.63 (PC6)
- net LED_R: now also D9.2 (A), U1.62 (PD15); no longer D8.2 (A), U1.66 (PC9)
- net UART3_RX: now also J1.3 (Pin_3); no longer J1.2 (Pin_2)
- net UART3_TX: now also J1.2 (Pin_2); no longer J1.3 (Pin_3)
- net at Q1.3 (C): now also LS1.P
- net at D8.1 (K): now also RN3.1 (R1.1)
- net at D4.1 (K): now also RN3.4 (R4.1)
- net at D9.1 (K): now also RN3.5 (R5.1)
- net at D5.1 (K): now also RN3.3 (R3.1)
- net at D3.1 (K): now also RN3.2 (R2.1)
Other:
- moved on the sheet: D3, D4, D8, D9
