File: schematic/_autosave-schematic.kicad_sch (KiCad schematic)
At the start: 79 parts, among them J1 Conn_01x04_Socket, J10 Conn_01x06_Pin, J11 Conn_01x06_Pin, J12 Conn_01x02_Socket, J2 Conn_01x04_Socket, J3 Conn_01x04_Socket, J4 Conn_01x04_Socket, J5 Conn_01x03_Pin, J6 Conn_01x03_Pin, J7 Conn_01x03_Pin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

Commit message: 1
Parts:
- removed J3: Conn_01x04_Socket, Connector_JST:JST_PH_B4B-PH-K_1x04_P2.00mm_Vertical, symbol Connector:Conn_01x04_Socket
- removed R12, R13, R14, R15, R16: 1K, Resistor_SMD:R_0603_1608Metric, symbol Device:R
- added C30, C31: 22uF, Capacitor_SMD:C_0201_0603Metric, symbol Device:C
- added R21: 1.1R, Resistor_SMD:R_0805_2012Metric, symbol Device:R
- added RN1: R_Network05, Resistor_SMD:R_Array_Convex_5x0603, symbol Device:R_Network05
- added RN2: R_Pack05, Resistor_SMD:R_Array_Convex_5x0603, symbol Device:R_Pack05
- added SW4: SW_DIP_x05, Button_Switch_SMD:SW_DIP_SPSTx05_Slide_KingTek_DSHP05TS_W7.62mm_P1.27mm, symbol Switch:SW_DIP_x05
- added U5: AMS1117-5.0, Package_TO_SOT_SMD:SOT-223-3_TabPin2, symbol Regulator_Linear:AMS1117-5.0
- J1, J4: footprint Connector_JST:JST_PH_B4B-PH-K_1x04_P2.00mm_Vertical -> Connector_PinHeader_2.54mm:PinHeader_1x04_P2.54mm_Vertical
- J10: footprint Connector_JST:JST_ZE_B06B-ZESK-D_1x06_P1.50mm_Vertical -> JST-254:JST 6
- J2: footprint Connector_JST:JST_PH_B4B-PH-K_1x04_P2.00mm_Vertical -> Connector_JST:JST_SH_BM04B-SRSS-TB_1x04-1MP_P1.00mm_Vertical
- J5, J6, J7, J8, J9: footprint Connector_JST:JST_PH_B3B-PH-K_1x03_P2.00mm_Vertical -> Connector_PinHeader_2.54mm:PinHeader_1x03_P2.54mm_Vertical
Connections:
- net +3V3: now also RN2.1 (R1.1), RN2.2 (R2.1), RN2.3 (R3.1), RN2.4 (R4.1), RN2.5 (R5.1)
- net +5V: now also C30.1, U5.2 (VO)
- net GND: now also C30.2, C31.2, RN1.1 (common), U5.1 (GND); no longer D3.1 (K), D4.1 (K), D5.1 (K), D6.1 (K), D7.1 (K)
- net LED_FF: now also D5.2 (A)
- net LED_FL: now also D3.2 (A)
- net LED_FR: now also D6.2 (A)
- net LED_L: now also D4.2 (A)
- net LED_R: now also D7.2 (A)
- net BIT_SW_4: now reaches U1.1 (PE2)
- net BIT_SW_4: now also SW4.6
- net BIT_SW_3: now reaches U1.2 (PE3)
- net BIT_SW_3: now also SW4.7
- net BIT_SW_2: now reaches U1.3 (PE4)
- net BIT_SW_2: now also SW4.8
- net BIT_SW_1: now reaches U1.4 (PE5)
- net BIT_SW_1: now also SW4.9
- net BIT_SW_0: now reaches U1.5 (PE6)
- net BIT_SW_0: now also SW4.10
- net UART1_RX: no longer names the net of U1.54 (PB15)
- net UART1_TX: no longer names the net of U1.53 (PB14)
- new net: D4.1 (K), RN1.2 (R1)
- new net: D3.1 (K), RN1.3 (R2)
- new net: D5.1 (K), RN1.4 (R3)
- new net: D6.1 (K), RN1.5 (R4)
- new net: D7.1 (K), RN1.6 (R5)
- new net: RN2.10 (R1.2), SW4.1
- new net: RN2.6 (R5.2), SW4.5
- new net: RN2.7 (R4.2), SW4.4
- new net: RN2.8 (R3.2), SW4.3
- new net: RN2.9 (R2.2), SW4.2
- new net: C31.1, R21.2, U5.3 (VI)
- new net +7.5V: R21.1
Other:
- note removed: "UART1"
- moved on the sheet: BZ1, C1, C10, C11, C12, C13, C14, C15, C16, C17, C18, C19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
