File: schematic/schematic.kicad_pcb (KiCad board)
At the start: 2 copper layers, 45 parts, among them J2 Conn_01x04_Socket, SW1 SW_Push, U1 STM32H743VITx, U2 AMS1117, U3 TB6612FNG_C_8_EL, U4 MP1584, Y1 Crystal_GND23_Small

Commit message: vẽ đủ đò ăn chơi chưa duyệt
Parts:
- added BZ1: Buzzer, Buzzer_Beeper:MagneticBuzzer_CUI_CMT-8504-100-SMT, F.Cu at (146.9, 123.0)
- added D2: LED, LED_SMD:LED_0603_1608Metric, F.Cu at (171.5, 89.5)
- added D3: LED, LED_SMD:LED_0603_1608Metric, F.Cu at (119.4, 70.8)
- added D4: LED, LED_SMD:LED_0603_1608Metric, F.Cu at (119.4, 73.3)
- added D5: LED, LED_SMD:LED_0603_1608Metric, F.Cu at (119.4, 75.9)
- added D6: LED, LED_SMD:LED_0603_1608Metric, F.Cu at (119.4, 78.5)
- added D7: LED, LED_SMD:LED_0603_1608Metric, F.Cu at (119.4, 81.1)
- added J1: Conn_01x04_Socket, Connector_JST:JST_PH_B4B-PH-K_1x04_P2.00mm_Vertical, F.Cu at (216.5, 107.5)
- added J10: Conn_01x06_Pin, Connector_JST:JST_PH_S6B-PH-K_1x06_P2.00mm_Horizontal, F.Cu at (202.8, 53.4)
- added J11: Conn_01x06_Pin, Connector_JST:JST_PH_S6B-PH-K_1x06_P2.00mm_Horizontal, F.Cu at (202.8, 63.0)
- added J3: Conn_01x04_Socket, Connector_JST:JST_PH_B4B-PH-K_1x04_P2.00mm_Vertical, F.Cu at (216.5, 114.0)
- added J4: Conn_01x04_Socket, Connector_JST:JST_PH_B4B-PH-K_1x04_P2.00mm_Vertical, F.Cu at (216.5, 120.6)
- added J5: Conn_01x03_Pin, Connector_JST:JST_PH_S3B-PH-K_1x03_P2.00mm_Horizontal, F.Cu at (204.5, 79.2)
- added J6: Conn_01x03_Pin, Connector_JST:JST_PH_S3B-PH-K_1x03_P2.00mm_Horizontal, F.Cu at (215.0, 79.3)
- added J7: Conn_01x03_Pin, Connector_JST:JST_PH_S3B-PH-K_1x03_P2.00mm_Horizontal, F.Cu at (226.5, 78.8)
- added J8: Conn_01x03_Pin, Connector_JST:JST_PH_B3B-PH-K_1x03_P2.00mm_Vertical, F.Cu at (205.8, 130.9)
- added J9: Conn_01x03_Pin, Connector_JST:JST_PH_B3B-PH-K_1x03_P2.00mm_Vertical, F.Cu at (205.8, 137.5)
- added Q1: S8550, Package_TO_SOT_SMD:SOT-23, F.Cu at (143.7, 130.9)
- added R10: 1K, Resistor_SMD:R_0603_1608Metric, F.Cu at (148.2, 129.8)
- added R11: 1K, Resistor_SMD:R_0603_1608Metric, F.Cu at (171.2, 93.0)
- added R12: 1K, Resistor_SMD:R_0603_1608Metric, F.Cu at (123.4, 70.7)
- added R13: 1K, Resistor_SMD:R_0603_1608Metric, F.Cu at (123.4, 73.2)
- added R14: 1K, Resistor_SMD:R_0603_1608Metric, F.Cu at (123.4, 75.7)
- added R15: 1K, Resistor_SMD:R_0603_1608Metric, F.Cu at (123.4, 78.2)
- added R16: 1K, Resistor_SMD:R_0603_1608Metric, F.Cu at (123.4, 80.8)
- Y1: footprint Crystal:Crystal_SMD_EuroQuartz_MJ-4Pin_5.0x3.2mm_HandSoldering -> Crystal:Crystal_SMD_3225-4Pin_3.2x2.5mm
- moved SW1 13.4 mm to (129.1, 135.0)
Connections:
- net Net-(U3-AO1@1) renamed /M1-R
- net Net-(U3-AO2@1) renamed /M1-L
- net Net-(U3-BO1@1) renamed /M2-R
- net Net-(U3-BO2@1) renamed /M2-L
- C22 pad 1: +3.3V -> +3V3
- C25 pad 1: +3.3V -> +3V3
- U1 pad 46: /UART3_TX -> /I2C2_SCL
- U1 pad 47: /UART3_RX -> /I2C2_SDA
- U1 pad 55: unconnected-(U1-PD8-Pad55) -> /UART3_TX
- U1 pad 56: unconnected-(U1-PD9-Pad56) -> /UART3_RX
- U1 pad 63: unconnected-(U1-PC6-Pad63) -> /LED_L
- U1 pad 64: unconnected-(U1-PC7-Pad64) -> /LED_R
- U1 pad 65: unconnected-(U1-PC8-Pad65) -> /LED_FL
- U1 pad 66: unconnected-(U1-PC9-Pad66) -> /LED_FR
- U1 pad 67: unconnected-(U1-PA8-Pad67) -> /LED_FF
- U1 pad 68: unconnected-(U1-PA9-Pad68) -> /BUZZ
- U3 pad 19: +3.3V -> +3V3
- U3 pad 20: +3.3V -> +3V3
