File: schematic/schematic.kicad_pcb (KiCad board)
At the start: 2 copper layers, 65 x 85 mm, 78 parts, among them J1 Conn_01x04_Socket, J10 Conn_01x06_Pin, J11 Conn_01x06_Pin, J2 Conn_01x04_Socket, J4 Conn_01x04_Socket, J5 Conn_01x07_Pin, Q1 S8550, SW1 SW_Push, SW2 SW_Push, SW3 SW_Push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

Commit message: thêm file thiet ke va da chinh sua nhung chua chot
Parts:
- moved C6 8.86 mm to (180.2, 87.5)
- moved C1 8.84 mm to (180.2, 85.8)
- moved C8 8.55 mm to (183.6, 92.6)
- moved C16 5.77 mm to (195.4, 86.6)
- moved Y1 5.77 mm to (195.4, 89.2)
- moved C17 5.77 mm to (195.4, 91.8)
- moved R4 4.90 mm to (182.7, 112.7)
- moved C18 4.90 mm to (184.3, 112.7)
- moved R7 4.72 mm to (167.6, 107.4), turned to 0 degrees
- moved R5 4.27 mm to (183.4, 109.7), turned to 180 degrees
- moved C32 3.22 mm to (183.4, 116.9)
- moved C3 1.93 mm to (183.7, 94.2)
- moved C7 1.59 mm to (183.6, 84.2)
- moved RN2 1.56 mm to (195.3, 94.8)
- moved C10 1.50 mm to (183.6, 85.9)
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- renumbered PIN to J12, SW1 to RESET
Connections:
- C18 pad 1: +5V -> +5VD
- C26 pad 1: +5V -> +5VD
- C27 pad 1: +5V -> +5VD
- C32 pad 1: +5V -> +5VD
- L1 pad 2: +5V -> +5VD
- R4 pad 1: +5V -> +5VD
- U3 pad 13: +5V -> +5VD
- U3 pad 14: +5V -> +5VD
- U3 pad 24: +5V -> +5VD
Routing:
- net +5V: track 109.5 -> 86.0 mm, vias 18 -> 3
- net +3V3: track 256.3 -> 276.5 mm, vias 15 -> 13
- net GND: track 7.75 -> 0.52 mm, vias 80 -> 77
- net /NRST: track 78.2 -> 85.0 mm
- net Net-(U4-FB): track 31.1 -> 25.9 mm
- net +5VD: track 0.00 -> 4.30 mm, vias 0 -> 24
- net /PH1: track 12.6 -> 8.59 mm
- net Net-(RN2-R4.2): track 3.17 -> 6.45 mm
- net Net-(RN2-R2.2): track 3.17 -> 6.42 mm
- net Net-(RN2-R5.2): track 3.42 -> 6.58 mm
- net Net-(RN2-R3.2): track 2.93 -> 6.06 mm
- net Net-(RN2-R1.2): track 3.40 -> 6.21 mm
- net /BUTTON_0: track 96.3 -> 94.4 mm
- net /PH0: track 10.5 -> 8.89 mm
- net /SWCLK: track 22.1 -> 23.6 mm
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- added copper zone on B.Cu, net +5VD
- added copper zone on F.Cu, net +5VD
- removed copper zone on B.Cu, net +5V
Other:
- board text added: "EN_A_L"
- board text added: "EN_A_R"
- board text added: "EN_B_L"
- board text added: "EN_B_R"
- board text added: "M+"
- board text added: "M-"
- board text added: "QUỶ ĐỎ 2 1112"
