File: schematic/schematic.kicad_pcb (KiCad board)
At the start: 2 copper layers, 65 x 85 mm, 78 parts, among them J1 Conn_01x04_Socket, J10 Conn_01x06_Pin, J11 Conn_01x06_Pin, J12 Conn_01x02_Socket, J2 Conn_01x04_Socket, J4 Conn_01x04_Socket, J5 Conn_01x07_Pin, Q1 S8550, SW2 SW_Push, SW3 SW_Push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

Commit message: đã đặt mạch
Parts:
- L1: value 15uH -> 22uH
- RN2: moved to F.Cu
- moter-r: renamed from J11; footprint Connector_JST:JST_SH_BM06B-SRSS-TB_1x06-1MP_P1.00mm_Vertical -> JST-254:JST 6
- motor-L: renamed from J10; footprint Connector_JST:JST_SH_BM06B-SRSS-TB_1x06-1MP_P1.00mm_Vertical -> JST-254:JST 6
- moved RN2 23.3 mm to (206.8, 74.6), turned to 180 degrees
- moved SW4 19.6 mm to (200.1, 74.7)
- moved moter-r 14.2 mm to (206.6, 104.5)
- moved motor-L 9.18 mm to (165.7, 109.9)
- moved C23 8.43 mm to (201.5, 113.8)
- moved C24 8.43 mm to (201.5, 111.6)
- moved R11 8.43 mm to (200.5, 109.5)
- moved D2 8.43 mm to (200.9, 106.7)
- moved U2 8.43 mm to (200.1, 111.6)
- moved C8 6.73 mm to (183.6, 85.9)
- moved C6 6.09 mm to (183.7, 92.5)
- moved C30 5.90 mm to (201.6, 117.4)
- moved C31 5.90 mm to (201.5, 122.0)
- moved R21 5.90 mm to (197.5, 124.9)
- moved U5 5.90 mm to (200.1, 119.6)
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- renumbered J2 to ST-LINK, J4 to i2c
Routing:
- net /BIT_SW_4: track 4.68 -> 41.8 mm, vias 0 -> 2
- net /BIT_SW_3: track 4.36 -> 41.1 mm, vias 0 -> 2
- net /BIT_SW_2: track 4.04 -> 40.6 mm, vias 0 -> 2
- net /BIT_SW_1: track 4.11 -> 39.6 mm, vias 0 -> 2
- net /BIT_SW_0: track 4.43 -> 39.1 mm, vias 0 -> 2
- net +3V3: track 276.5 -> 290.3 mm
- net 6.5-7.5V: track 49.9 -> 41.0 mm
- net /EN_A_R: track 28.7 -> 21.7 mm
- net /EN_B_R: track 30.4 -> 23.7 mm
- net Net-(D1-K): track 9.29 -> 2.88 mm
- net /NRST: track 85.0 -> 79.8 mm
- net Net-(RN2-R4.2): track 6.45 -> 2.23 mm, vias 1 -> 0
- net Net-(RN2-R5.2): track 6.58 -> 2.45 mm, vias 1 -> 0
- net Net-(RN2-R2.2): track 6.42 -> 2.36 mm, vias 1 -> 0
- net Net-(RN2-R3.2): track 6.06 -> 2.10 mm, vias 1 -> 0
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Other:
- board text added: "G"

Commit message: thư viện đọc sensor analog
Parts:
- turned Q1 to 0 degrees
- renumbered LS1 to BUZZER
Changed lines of the file:
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@@
 	(footprint "Package_TO_SOT_SMD:SOT-23"
 		(layer "F.Cu")
-		(at 158 74.1 90)
+		(at 157.992163 74.090219)
 		(descr "SOT, 3 Pin (https://www.jedec.org/system/files/docs/to-236h.pdf variant AB), generated with kicad-footprint-generator ipc_gullwing_generator.py")
 		(tags "SOT TO_SOT_SMD")
 		(property "Reference" "Q1"
-			(at 0 -2.4 90)
+			(at -2.2 0.2 90)
 			(layer "F.SilkS")
 			(hide yes)
@@
 		)
 		(property "Value" "S8550"
-			(at 0.4 -2.4 90)
+			(at -2.2 -0.2 90)
 			(layer "F.Fab")
 			(hide yes)
@@
 		)
 		(property "Footprint" "Package_TO_SOT_SMD:SOT-23"
-			(at 0.4 0 -90)
+			(at 0.2 -0.2 -90)
 			(unlocked yes)
 			(layer "F.Fab")
@@
 		)
 		(property "Datasheet" "http://www.unisonic.com.tw/datasheet/S8550.pdf"
-			(at 0.4 0 -90)
+			(at 0.2 -0.2 -90)
 			(unlocked yes)
 			(layer "F.Fab")
@@
 		)
 		(property "Description" "0.7A Ic, 20V Vce, Low Voltage High Current PNP Transistor, TO-92"
-			(at 0.4 0 -90)
+			(at 0.2 -0.2 -90)
 			(unlocked yes)
 			(layer "F.Fab")
@@
 		(attr smd)
 		(fp_line
-			(start 0.4 -1.56)
-			(end 1.05 -1.56)
+			(start -1.36 -0.2)
+			(end -1.36 -0.85)
 			(stroke
 				(width 0.12)
@@
 		)
 		(fp_line
-			(start 0.4 -1.56)
-			(end -0.25 -1.56)
+			(start -1.36 -0.2)
+			(end -1.36 0.45)
 			(stroke
 				(width 0.12)
@@
 		)
 		(fp_line
-			(start 0 -1.56)
-			(end 0.65 -1.56)
+			(start -1.36 0.2)
+			(end -1.36 -0.45)
 			(stroke
 				(width 0.12)
@@
 		)
 		(fp_line
-			(start 0 -1.56)
-			(end -0.65 -1.56)
+			(start -1.36 0.2)
+			(end -1.36 0.85)
 			(stroke
 				(width 0.12)
@@
 		(fp_poly
 			(pts
-				(xy -1.1625 -1.51) (xy -1.4025 -1.84) (xy -0.9225 -1.84) (xy -1.1625 -1.51)
+				(xy -1.31 1.3625) (xy -1.64 1.6025) (xy -1.64 1.1225) (xy -1.31 1.3625)
 			)
 			(stroke
@@
 		)
 		(fp_line
-			(start 2.32 -1.7)
-			(end -1.52 -1.7)
+			(start -1.5 -2.15)
+			(end -1.5 1.72)
 			(stroke
 				(width 0.05)
@@
 		)
 		(fp_line
-			(start 1.92 -1.7)
-			(end -1.92 -1.7)
+			(start -1.5 -2.15)
+			(end 1.9 -2.15)
 			(stroke
 				(width 0.05)
@@
 		)
 		(fp_line
-			(start -1.52 -1.7)
-			(end -1.52 1.7)
+			(start -1.5 -1.72)
+			(end -1.5 2.12)
 			(stroke
 				(width 0.05)
@@
 		)
 		(fp_line
-			(start -1.92 -1.7)
-			(end -1.92 1.7)
+			(start -1.5 1.72)
+			(end 1.9 1.72)
 			(stroke
 				(width 0.05)
@@
 		)
 		(fp_line
-			(start 1.05 -1.45)
-			(end 1.05 1.125)
+			(start -1.5 2.12)
+			(end 1.9 2.12)
 			(stroke
-				(width 0.1)
+				(width 0.05)
 				(type solid)
 			)
-			(layer "F.Fab")
+			(layer "F.CrtYd")
+		)
+		(fp_line
+			(start 1.9 -2.15)
+			(end 1.9 1.69)
+			(stroke
+				(width 0.05)
+				(type solid)
+			)
+			(layer "F.CrtYd")
 		)
 		(fp_line
-			(start -0.25 -1.45)
-			(end 1.05 -1.45)
+			(start 1.9 -1.74)
+			(end 1.9 2.1)
+			(stroke
+				(width 0.05)
+				(type solid)
+			)
+			(layer "F.CrtYd")
+		)
+		(fp_line
+			(start -1.25 -0.85)
+			(end 1.325 -0.85)
 			(stroke
 				(width 0.1)
@@
 		)
 		(fp_line
-			(start -0.325 -1.45)
-			(end 0.65 -1.45)
+			(start -1.25 0.45)
+			(end -1.25 -0.85)
 			(stroke
 				(width 0.1)
@@
 		)
 		(fp_line
-			(start -0.65 -1.125)
-			(end -0.325 -1.45)
+			(start -1.25 0.525)
+			(end -1.25 -0.45)
 			(stroke
 				(width 0.1)
@@
 		)
 		(fp_line
-			(start -0.25 1.45)
-			(end -0.25 -1.45)
+			(start -0.925 0.85)
+			(end -1.25 0.525)
 			(stroke
 				(width 0.1)
@@
 			(layer "F.Fab")
 		)
-		(fp_text user "${REFERENCE}"
-			(at 0.4 0 90)
-			(layer "F.Fab")
-			(effects
-				(font
-					(size 0.32 0.32)
-					(thickness 0.05)
-				)
+		(fp_line
+			(start 1.65 0.45)
+			(end -1.25 0.45)
+			(stroke
+				(width 0.1)
+				(type solid)
 			)
+			(layer "F.Fab")
 		)
 		(pad "1" smd rect
-			(at 1.3375 -0.95 270)
+			(at -0.75 -1.1375 270)
 			(size 1.475 0.6)
 			(layers "F.Cu" "F.Paste" "F.Mask")
@@
 		)
 		(pad "2" smd rect
-			(at 1.3375 0.95 270)
+			(at 1.15 -1.1375 270)
 			(size 1.475 0.6)
 			(layers "F.Cu" "F.Paste" "F.Mask")
@@
 		)
 		(pad "3" smd rect
-			(at -0.5375 0 270)
+			(at 0.2 0.7375 270)
 			(size 1.475 0.6)
 			(layers "F.Cu" "F.Paste" "F.Mask")
@@
 		(model "${KICAD8_3DMODEL_DIR}/Package_TO_SOT_SMD.3dshapes/SOT-23.wrl"
 			(offset
-				(xyz 0 0 0)
+				(xyz 0.2 0 0)
 			)
 			(scale
@@
 			)
 			(rotate
-				(xyz 0 0 0)
+				(xyz 0 0 90)
 			)
 		)
@@
 		(layer "F.Cu")
 		(at 157.022163 65.720219)
-		(property "Reference" "LS1"
+		(property "Reference" "BUZZER"
 			(at 0 0 90)
 			(layer "F.SilkS")
@@
 		)
 		(property "Footprint" "JST-254:JST 6"
-			(at 0 0 360)
+			(at 0 0 0)
 			(layer "B.Fab")
 			(hide yes)
@@
 		)
 		(property "Datasheet" ""
-			(at 0 0 360)
+			(at 0 0 0)
 			(layer "B.Fab")
 			(hide yes)
@@
 		)
 		(property "Description" "Generic connector, single row, 01x06, script generated"
-			(at 0 0 360)
+			(at 0 0 0)
 			(layer "B.Fab")
 			(hide yes)
@@
 	)
 	(segment
+		(start 157.65 77.925)
+		(end 157.65 76.738056)
+		(width 0.5)
+		(layer "F.Cu")
+		(net 63)
+	)
+	(segment
 		(start 187.752163 104.070219)
 		(end 187.752163 96.870219)
@@
 	)
 	(segment
-		(start 157.65 77.925)
-		(end 157.65 76.738056)
-		(width 0.5)
-		(layer "F.Cu")
-		(net 63)
-	)
-	(segment
 		(start 204.082163 110.810219)
 		(end 204.082163 101.960219)
@@
 	)
 	(segment
-		(start 157.65 76.738056)
-		(end 157.05 76.138056)
-		(width 0.5)
-		(layer "F.Cu")
-		(net 63)
-	)
-	(segment
 		(start 152.38 83.6)
 		(end 150.391944 83.6)
@@
 	)
 	(segment
+		(start 157.232163 76.320219)
+		(end 157.232163 72.962719)
+		(width 0.5)
+		(layer "F.Cu")
+		(net 63)
+	)
+	(segment
 		(start 186.111944 92.5)
 		(end 187.475 92.5)
@@
 	)
 	(segment
+		(start 157.232163 72.962719)
+		(end 157.242163 72.952719)
+		(width 0.5)
+		(layer "F.Cu")
+		(net 63)
+	)
+	(segment
 		(start 185.352163 89)
 		(end 185.352163 89.580219)
@@
 	)
 	(segment
-		(start 157.05 76.138056)
-		(end 157.05 72.7625)
-		(width 0.5)
-		(layer "F.Cu")
-		(net 63)
-	)
-	(segment
 		(start 150.372163 80.000219)
 		(end 152.447382 77.925)
@@
 	)
 	(segment
+		(start 157.65 76.738056)
+		(end 157.232163 76.320219)
+		(width 0.5)
+		(layer "F.Cu")
+		(net 63)
+	)
+	(segment
 		(start 202.692163 111.000219)
 		(end 203.292163 111.600219)
@@
 	)
 	(segment
-		(start 158.95 72.7625)
-		(end 159.157719 72.970219)
-		(width 0.3)
-		(layer "F.Cu")
-		(net 91)
-	)
-	(segment
-		(start 159.157719 72.970219)
-		(end 160.970219 72.970219)
+		(start 161.039781 73.060219)
+		(end 161.05 73.05)
 		(width 0.3)
 		(layer "F.Cu")
@@
 	)
 	(segment
-		(start 159.0375 73.05)
-		(end 158.9375 73.15)
+		(start 159.249663 73.060219)
+		(end 161.039781 73.060219)
 		(width 0.3)
 		(layer "F.Cu")
@@
 	)
 	(segment
-		(start 160.970219 72.970219)
-		(end 161.05 73.05)
+		(start 159.142163 72.952719)
+		(end 159.249663 73.060219)
 		(width 0.3)
 		(layer "F.Cu")
@@
 	)
 	(segment
-		(start 158 69.982382)
+		(start 158.192163 74.827719)
+		(end 158.172163 74.807719)
+		(width 0.3)
+		(layer "F.Cu")
+		(net 115)
+	)
+	(segment
+		(start 158.172163 69.810219)
 		(end 158.762163 69.220219)
 		(width 0.3)
@@
 	)
 	(segment
-		(start 158 74.6375)
-		(end 158 69.982382)
+		(start 158.172163 74.807719)
+		(end 158.172163 69.810219)
 		(width 0.3)
 		(layer "F.Cu")
